Commit message: Fix *.stl file path

File: screw_tool/urdf/screw_tool.urdf (robot description, URDF)
Before this commit: robot screw_tool, 1 links, 0 joints
Links:
- link screw_tool: geometry collision mesh filename=$(find rl_gazebo_sim)/screw_tool/meshes/screw_tool.STL; visual mesh filename=$(find rl_gazebo_sim)/screw_tool/meshes/screw_tool.STL
