Commit message: fixed tool paths and finished conecting dummy tool

File: ur5_robot_w_tool/ur5_robot_w_tool.urdf.xacro (robot description, xacro)
@@ -6,10 +6,10 @@
   <!-- ur5 -->
   <xacro:include filename="$(find ur_description)/urdf/ur5.urdf.xacro" />
-  <!-- tool
-  <xacro:include filename="$(find rl_simulation)/screw_tool/urdf/screw_tool.urdf" />
--->
+  <!-- tool -->
+  <xacro:include filename="$(find rl_gazebo_sim)/screw_tool/urdf/screw_tool.urdf" />
   <!-- arm -->
   <xacro:ur5_robot prefix="" joint_limited="false"/>
   <link name="world" />
+  <!-- fix the arm in the world -->
   <joint name="world_joint" type="fixed">
     <parent link="world" />
@@ -17,11 +17,11 @@
     <origin xyz="0.0 0.0 0.0" rpy="0.0 0.0 0.0" />
   </joint>
-   <!--
-  <link name="screw_tool" />
-  <joint name="tool0-screw_tool" type="fixed">
+  <!-- tool -->
+  <!-- give it a name and type -->
+  <!-- add the tool to the end-effector -->
+  <joint name="screw_tool_joint" type="fixed">
     <parent link="tool0" />
     <child link="screw_tool" />
     <origin xyz="0 0 0" rpy="0 0 0" />
   </joint>
-  -->
 </robot>

Commit message: still trying to add ft sensor to robot

File: ur5_robot_w_tool/ur5_robot_w_tool.urdf.xacro (robot description, xacro)
@@ -20,8 +20,22 @@
   <!-- give it a name and type -->
   <!-- add the tool to the end-effector -->
-  <joint name="screw_tool_joint" type="fixed">
+  <joint name="screw_tool_joint" type="revolute">
     <parent link="tool0" />
     <child link="screw_tool" />
-    <origin xyz="0 0 0" rpy="0 0 0" />
+    <origin xyz="0 0 0.1" rpy="0 0 0" />
+    <limit velocity="6.5" effort="1000" lower="0" upper="0" />  <!--This is a bugfix. Using fixed type joint causes problems with FT-sensor.-->
   </joint>
+  <!-- Activate the feedback
+  <gazebo reference="wrist_3_link-tool0_fixed_joint">
+    <provideFeedback>true</provideFeedback>
+  </gazebo>-->
+  <!-- FT sensor
+  <gazebo>
+    <plugin name="FTsensor_controller"    filename="libgazebo_ros_ft_sensor.so">
+       <updateRate>100.0</updateRate>
+       <topicName>FTsensor_topic</topicName>
+       <gaussianNoise>0.0</gaussianNoise>
+       <jointName>wrist_3_link-tool0_fixed_joint</jointName>
+    </plugin>
+  </gazebo>-->
 </robot>

Commit message: added force torque sensor on dummy tool

File: ur5_robot_w_tool/ur5_robot_w_tool.urdf.xacro (robot description, xacro)
@@ -1,3 +1,3 @@
-<?xml version="1.0"?>
+<?xml version="2.0"?>
 <robot xmlns:xacro="http://ros.org/wiki/xacro"
        name="ur5" >
@@ -7,7 +7,9 @@
   <xacro:include filename="$(find ur_description)/urdf/ur5.urdf.xacro" />
   <!-- tool -->
-  <xacro:include filename="$(find rl_gazebo_sim)/screw_tool/urdf/screw_tool.urdf" />
+  <xacro:include filename="$(find rl_gazebo_sim)/screw_tool/urdf/screw_tool.urdf.xacro" />
   <!-- arm -->
   <xacro:ur5_robot prefix="" joint_limited="false"/>
+  <!-- tool -->
+  <xacro:my_tool parrent_link="wrist_3_link" origin_xyz="0 0.0823 0" origin_rpy="${pi/-2.0} 0 0"/>
   <link name="world" />
   <!-- fix the arm in the world -->
@@ -17,25 +19,3 @@
     <origin xyz="0.0 0.0 0.0" rpy="0.0 0.0 0.0" />
   </joint>
-  <!-- tool -->
-  <!-- give it a name and type -->
-  <!-- add the tool to the end-effector -->
-  <joint name="screw_tool_joint" type="revolute">
-    <parent link="tool0" />
-    <child link="screw_tool" />
-    <origin xyz="0 0 0.1" rpy="0 0 0" />
-    <limit velocity="6.5" effort="1000" lower="0" upper="0" />  <!--This is a bugfix. Using fixed type joint causes problems with FT-sensor.-->
-  </joint>
-  <!-- Activate the feedback
-  <gazebo reference="wrist_3_link-tool0_fixed_joint">
-    <provideFeedback>true</provideFeedback>
-  </gazebo>-->
-  <!-- FT sensor
-  <gazebo>
-    <plugin name="FTsensor_controller"    filename="libgazebo_ros_ft_sensor.so">
-       <updateRate>100.0</updateRate>
-       <topicName>FTsensor_topic</topicName>
-       <gaussianNoise>0.0</gaussianNoise>
-       <jointName>wrist_3_link-tool0_fixed_joint</jointName>
-    </plugin>
-  </gazebo>-->
 </robot>
