Commit message: added the real ft sensor, thoug it's misalligned

File: rl_gazebo_sim/ur5_robot_w_tool/ur5_robot_w_tool.urdf.xacro (robot description, xacro)
@@ -7,9 +7,9 @@
   <xacro:include filename="$(find ur_description)/urdf/ur5.urdf.xacro" />
   <!-- tool -->
-  <xacro:include filename="$(find rl_gazebo_sim)/screw_tool/urdf/screw_tool.urdf.xacro" />
+  <xacro:include filename="$(find rl_gazebo_sim)/screw_tool/screw_tool.urdf.xacro" />
   <!-- arm -->
   <xacro:ur5_robot prefix="" joint_limited="false"/>
   <!-- tool -->
-  <xacro:my_tool parrent_link="wrist_3_link" origin_xyz="0 0.0823 0" origin_rpy="${pi/-2.0} 0 0"/>
+  <xacro:my_tool parrent_link="wrist_3_link" origin_xyz="0 0.0823 0" origin_rpy="0 0 0"/>
   <link name="world" />
   <!-- fix the arm in the world -->

File: rl_gazebo_sim/urdf/DrillAndMountAssembly.urdf (robot description, URDF)
Before this commit: robot DrillAndMountAssembly, 1 links, 0 joints
Links:
- link DrillAndMountAssembly: geometry collision mesh filename=$(find rl_gazebo_sim)/meshes/DrillAndMountAssembly.STL; visual mesh filename=$(find rl_gazebo_sim)/meshes/DrillAndMountAssembly.STL

File: rl_gazebo_sim/urdf/ForceTorqueWithMount.urdf (robot description, URDF)
Before this commit: robot ForceTorqueWithMount, 1 links, 0 joints
Links:
- link ForceTorqueWithMount: geometry collision mesh filename=$(find rl_gazebo_sim)/meshes/ForceTorqueWithMount.STL; visual mesh filename=$(find rl_gazebo_sim)/meshes/ForceTorqueWithMount.STL
