Commit message: added the screw machine to the robot, but it's  not alligned in stl file

File: rl_gazebo_sim/screw_tool/screw_tool.urdf.xacro (robot description, xacro)
@@ -10,6 +10,6 @@
       <child link="ForceTorqueWithMount"/>
       <axis xyz="0.0 0.0 1.0"/>
-       <limit velocity="6.5" effort="1000" lower="0" upper="0" />  <!--This is a bugfix. Using fixed type joint causes problems with FT-sensor.-->
-    </joint>>
+      <limit velocity="6.5" effort="1000" lower="0" upper="0" />  <!--This is a bugfix. Using fixed type joint causes problems with FT-sensor.-->
+    </joint>
     <!-- Activate the feedback -->
     <gazebo reference="${parrent_link}-ForceTorqueWithMount">
@@ -25,6 +25,14 @@
       </plugin>
     </gazebo>
-    <!-- Drill and mount
-    <xacro:macro filename="$(find rl_gazebo_sim)/urdf/DrillAndMountAssembly.urdf"/>-->
+    <!-- Drill and mount -->
+    <xacro:include filename="$(find rl_gazebo_sim)/urdf/DrillAndMountAssembly.urdf"/>
+    <!-- Add the drill to the chain -->
+    <joint name="ForceTorqueWithMount-DrillAndMountAssembly" type="fixed">
+      <origin xyz="0.0 0.0 0.0" rpy="0.0 0.0 0.0"/>
+      <parent link="ForceTorqueWithMount"/>
+      <child link="DrillAndMountAssembly"/>
+      <axis xyz="0.0 0.0 0.0"/>
+      <limit lower="0.0" upper="0.0" effort="0.0" velocity="0.0"/>
+    </joint>
   </xacro:macro>
 </robot>

File: rl_gazebo_sim/ur5_robot_w_tool/ur5_robot_w_tool.urdf.xacro (robot description, xacro)
@@ -11,5 +11,5 @@
   <xacro:ur5_robot prefix="" joint_limited="false"/>
   <!-- tool -->
-  <xacro:my_tool parrent_link="wrist_3_link" origin_xyz="0 0.0823 0" origin_rpy="0 0 0"/>
+  <xacro:my_tool parrent_link="wrist_3_link" origin_xyz="0 0.0823 0" origin_rpy="${pi/-2.0} ${pi/-2.0} ${pi/-2.0}"/>
   <link name="world" />
   <!-- fix the arm in the world -->

Commit message: added the tool. missing the screw bitz

File: rl_gazebo_sim/screw_tool/screw_tool.urdf.xacro (robot description, xacro)
@@ -29,5 +29,5 @@
     <!-- Add the drill to the chain -->
     <joint name="ForceTorqueWithMount-DrillAndMountAssembly" type="fixed">
-      <origin xyz="0.0 0.0 0.0" rpy="0.0 0.0 0.0"/>
+      <origin xyz="0 -0.06342 0" rpy="0.0 ${pi/4} 0.0"/>
       <parent link="ForceTorqueWithMount"/>
       <child link="DrillAndMountAssembly"/>
@@ -35,4 +35,14 @@
       <limit lower="0.0" upper="0.0" effort="0.0" velocity="0.0"/>
     </joint>
-  </xacro:macro>
+    <!-- include the screw bit-->
+    <xacro:include filename="$(find rl_gazebo_sim)/urdf/ScrewDriverBitStar.urdf"/>
+    <!-- add the screw bit to the screw machine-->
+    <joint name="DrillAndMountAssembly-ScrewDriverBitStar" type="revolute">
+      <origin xyz="0.0 -0.157 0.0" rpy="0.0 0.0 0.0"/>
+      <parent link="DrillAndMountAssembly"/>
+      <child link="ScrewDriverBitStar"/>
+      <axis xyz="0.0 0.0 1"/>
+      <limit effort="0.0" velocity="0.0"/>
+    </joint>
+  </xacro:macro>  0.0
 </robot>

File: rl_gazebo_sim/ur5_robot_w_tool/ur5_robot_w_tool.urdf.xacro (robot description, xacro)
@@ -11,5 +11,5 @@
   <xacro:ur5_robot prefix="" joint_limited="false"/>
   <!-- tool -->
-  <xacro:my_tool parrent_link="wrist_3_link" origin_xyz="0 0.0823 0" origin_rpy="${pi/-2.0} ${pi/-2.0} ${pi/-2.0}"/>
+  <xacro:my_tool parrent_link="wrist_3_link" origin_xyz="0 0.0823 0" origin_rpy="${pi} ${pi/4} 0"/>
   <link name="world" />
   <!-- fix the arm in the world -->

File: rl_gazebo_sim/urdf/ScrewDriverBitStar.urdf (robot description, URDF)
Before this commit: robot ScrewDriverBitStar, 1 links, 0 joints
Links:
- link ScrewDriverBitStar: geometry collision mesh filename=$(find rl_gazebo_sim)/meshes/ScrewDriverBitStar.STL; visual mesh filename=$(find rl_gazebo_sim)/meshes/ScrewDriverBitStar.STL

Commit message: cannot add the screwDriverBitStar to the model

File: rl_gazebo_sim/screw_tool/screw_tool.urdf.xacro (robot description, xacro)
@@ -25,7 +25,7 @@
       </plugin>
     </gazebo>
-    <!-- Drill and mount -->
-    <xacro:include filename="$(find rl_gazebo_sim)/urdf/DrillAndMountAssembly.urdf"/>
-    <!-- Add the drill to the chain -->
+    <!-- Drill and mount
+    <xacro:include filename="$(find rl_gazebo_sim)/urdf/DrillAndMountAssembly.urdf"/> -->
+    <!-- Add the drill to the chain
     <joint name="ForceTorqueWithMount-DrillAndMountAssembly" type="fixed">
       <origin xyz="0 -0.06342 0" rpy="0.0 ${pi/4} 0.0"/>
@@ -34,13 +34,13 @@
       <axis xyz="0.0 0.0 0.0"/>
       <limit lower="0.0" upper="0.0" effort="0.0" velocity="0.0"/>
-    </joint>
+    </joint>-->
     <!-- include the screw bit-->
     <xacro:include filename="$(find rl_gazebo_sim)/urdf/ScrewDriverBitStar.urdf"/>
     <!-- add the screw bit to the screw machine-->
-    <joint name="DrillAndMountAssembly-ScrewDriverBitStar" type="revolute">
-      <origin xyz="0.0 -0.157 0.0" rpy="0.0 0.0 0.0"/>
-      <parent link="DrillAndMountAssembly"/>
+    <joint name="ForceTorqueWithMount-ScrewDriverBitStar" type="revolute">
+      <origin xyz="0.0 -0.09358 0.0" rpy="0.0 0.0 0.0"/>
+      <parent link="ForceTorqueWithMount"/>
       <child link="ScrewDriverBitStar"/>
-      <axis xyz="0.0 0.0 1"/>
+      <axis xyz="1 0 0"/>
       <limit effort="0.0" velocity="0.0"/>
     </joint>

Commit message: bug: making joints reqolute makes them dissaper without any warnings or errors

File: rl_gazebo_sim/screw_tool/screw_tool.urdf.xacro (robot description, xacro)
@@ -25,7 +25,7 @@
       </plugin>
     </gazebo>
-    <!-- Drill and mount
-    <xacro:include filename="$(find rl_gazebo_sim)/urdf/DrillAndMountAssembly.urdf"/> -->
-    <!-- Add the drill to the chain
+    <!-- Drill and mount -->
+    <xacro:include filename="$(find rl_gazebo_sim)/urdf/DrillAndMountAssembly.urdf"/>
+    <!-- Add the drill to the chain -->
     <joint name="ForceTorqueWithMount-DrillAndMountAssembly" type="fixed">
       <origin xyz="0 -0.06342 0" rpy="0.0 ${pi/4} 0.0"/>
@@ -34,15 +34,14 @@
       <axis xyz="0.0 0.0 0.0"/>
       <limit lower="0.0" upper="0.0" effort="0.0" velocity="0.0"/>
-    </joint>-->
+    </joint>
     <!-- include the screw bit-->
     <xacro:include filename="$(find rl_gazebo_sim)/urdf/ScrewDriverBitStar.urdf"/>
     <!-- add the screw bit to the screw machine-->
     <joint name="ForceTorqueWithMount-ScrewDriverBitStar" type="revolute">
-      <origin xyz="0.0 -0.09358 0.0" rpy="0.0 0.0 0.0"/>
+      <origin xyz="0 -0.19652 0" rpy="0 0 0" />
       <parent link="ForceTorqueWithMount"/>
       <child link="ScrewDriverBitStar"/>
-      <axis xyz="1 0 0"/>
-      <limit effort="0.0" velocity="0.0"/>
-    </joint>
-  </xacro:macro>  0.0
+      <axis xyz="0.0 0.0 1.0"/>
+      <limit velocity="6.5" effort="1000" lower="0" upper="0" />     </joint>
+  </xacro:macro>
 </robot>

Commit message: tool fully assembled and mounted on robot

File: rl_gazebo_sim/screw_tool/screw_tool.urdf.xacro (robot description, xacro)
@@ -39,9 +39,10 @@
     <!-- add the screw bit to the screw machine-->
     <joint name="ForceTorqueWithMount-ScrewDriverBitStar" type="revolute">
-      <origin xyz="0 -0.19652 0" rpy="0 0 0" />
+      <origin xyz="0 -0.22042 0" rpy="0 0 0" /> <!--sunken 5mm in to the bit holder -->
       <parent link="ForceTorqueWithMount"/>
       <child link="ScrewDriverBitStar"/>
-      <axis xyz="0.0 0.0 1.0"/>
-      <limit velocity="6.5" effort="1000" lower="0" upper="0" />     </joint>
+      <axis xyz="0 1 0"/>
+      <limit velocity="1000" effort="1" lower="-1e+16" upper="1e+16"/>
+      </joint>
   </xacro:macro>
 </robot>

File: rl_gazebo_sim/urdf/ScrewDriverBitStar.urdf (robot description, URDF)
Before this commit: robot ScrewDriverBitStar, 1 links, 0 joints
Links:
- link ScrewDriverBitStar: mass 0 -> 0.01

Commit message: added autogenerated movit config package

File: rl_gazebo_sim/screw_tool/screw_tool.urdf.xacro (robot description, xacro)
@@ -43,5 +43,5 @@
       <child link="ScrewDriverBitStar"/>
       <axis xyz="0 1 0"/>
-      <limit velocity="1000" effort="1" lower="-1e+16" upper="1e+16"/>
+      <limit velocity="1000" effort="1" lower="-100000000" upper="100000000"/>
       </joint>
   </xacro:macro>

File: rl_gazebo_sim/urdf/DrillAndMountAssembly.urdf (robot description, URDF)
Before this commit: robot DrillAndMountAssembly, 1 links, 0 joints
Links:
- link DrillAndMountAssembly: geometry collision mesh filename=package://rl_gazebo_sim/meshes/DrillAndMountAssembly.STL; visual mesh filename=package://rl_gazebo_sim/meshes/DrillAndMountAssembly.STL

File: rl_gazebo_sim/urdf/ForceTorqueWithMount.urdf (robot description, URDF)
Before this commit: robot ForceTorqueWithMount, 1 links, 0 joints
Links:
- link ForceTorqueWithMount: geometry collision mesh filename=package://rl_gazebo_sim/meshes/ForceTorqueWithMount.STL; visual mesh filename=package://rl_gazebo_sim/meshes/ForceTorqueWithMount.STL

File: rl_gazebo_sim/urdf/ScrewDriverBitStar.urdf (robot description, URDF)
Before this commit: robot ScrewDriverBitStar, 1 links, 0 joints
Links:
- link ScrewDriverBitStar: geometry collision mesh filename=package://rl_gazebo_sim/meshes/ScrewDriverBitStar.STL; visual mesh filename=package://rl_gazebo_sim/meshes/ScrewDriverBitStar.STL

Commit message: update to the moveit config package because of a name conflict

File: rl_gazebo_sim/screw_tool/screw_tool.urdf.xacro (robot description, xacro)
@@ -5,5 +5,5 @@
     <xacro:include filename="$(find rl_gazebo_sim)/urdf/ForceTorqueWithMount.urdf"/>
     <!-- add the ft-senser -->
-    <joint name="${parrent_link}-ForceTorqueWithMount" type="revolute">
+    <joint name="${parrent_link}_ForceTorqueWithMount" type="revolute">
       <origin xyz="${origin_xyz}" rpy="${origin_rpy}" />
       <parent link="${parrent_link}"/>
@@ -13,5 +13,5 @@
     </joint>
     <!-- Activate the feedback -->
-    <gazebo reference="${parrent_link}-ForceTorqueWithMount">
+    <gazebo reference="${parrent_link}_ForceTorqueWithMount">
       <provideFeedback>true</provideFeedback>
     </gazebo>
@@ -22,5 +22,5 @@
         <topicName>FTsensor_topic</topicName>
         <gaussianNoise>0.0</gaussianNoise>
-        <jointName>${parrent_link}-ForceTorqueWithMount</jointName>
+        <jointName>${parrent_link}_ForceTorqueWithMount</jointName>
       </plugin>
     </gazebo>
@@ -28,5 +28,5 @@
     <xacro:include filename="$(find rl_gazebo_sim)/urdf/DrillAndMountAssembly.urdf"/>
     <!-- Add the drill to the chain -->
-    <joint name="ForceTorqueWithMount-DrillAndMountAssembly" type="fixed">
+    <joint name="ForceTorqueWithMount_DrillAndMountAssembly" type="fixed">
       <origin xyz="0 -0.06342 0" rpy="0.0 ${pi/4} 0.0"/>
       <parent link="ForceTorqueWithMount"/>
@@ -38,5 +38,5 @@
     <xacro:include filename="$(find rl_gazebo_sim)/urdf/ScrewDriverBitStar.urdf"/>
     <!-- add the screw bit to the screw machine-->
-    <joint name="ForceTorqueWithMount-ScrewDriverBitStar" type="revolute">
+    <joint name="ForceTorqueWithMount_ScrewDriverBitStar" type="revolute">
       <origin xyz="0 -0.22042 0" rpy="0 0 0" /> <!--sunken 5mm in to the bit holder -->
       <parent link="ForceTorqueWithMount"/>

Commit message: controller still not working

File: rl_gazebo_sim/screw_tool/screw_tool.urdf.xacro (robot description, xacro)
@@ -45,4 +45,11 @@
       <limit velocity="1000" effort="1" lower="-100000000" upper="100000000"/>
       </joint>
+    <!-- Frame coincident with all-zeros TCP on UR controller -->
+    <link name="ee_tip"/>
+    <joint name="ScrewDriverBitStar_ee_tip" type="fixed">
+      <origin xyz="0 -0.025 0" rpy="${pi/-2.0} 0 0"/>
+      <parent link="ScrewDriverBitStar"/>
+      <child link="ee_tip"/>
+    </joint>
   </xacro:macro>
 </robot>
