Commit message: renamed for easier readability. Rotation also changed to 0  instad of pi/2

File: rl_gazebo_sim/parts_descriptions/urdf/drill.urdf (robot description, URDF)
Before this commit: robot DrillAndMountAssembly, 1 links, 0 joints
Links:
- removed link DrillAndMountAssembly
- added link drill, mass 0.8; collision mesh filename=package://rl_gazebo_sim/parts_descriptions/meshes/drill.STL; visual mesh filename=package://rl_gazebo_sim/parts_descriptions/meshes/drill.STL

File: rl_gazebo_sim/parts_descriptions/urdf/ft_sensor.urdf (robot description, URDF)
Before this commit: robot ForceTorqueWithMount, 1 links, 0 joints
Links:
- removed link ForceTorqueWithMount
- added link ft_sensor, mass 1; collision mesh filename=package://rl_gazebo_sim/parts_descriptions/meshes/ft_sensor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; visual mesh filename=package://rl_gazebo_sim/parts_descriptions/meshes/ft_sensor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
