Commit message: cleanup

File: rl_gazebo_sim/parts_descriptions/urdf/CompleteToolAssembly.urdf (robot description, URDF)
Before this commit: robot CompleteToolAssembly, 1 links, 0 joints
Links:
- link CompleteToolAssembly: geometry collision mesh filename=package://rl_gazebo_sim/parts_descriptions/meshes/CompleteT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; visual mesh filename=package://rl_gazebo_sim/parts_descriptions/meshes/CompleteT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

File: rl_gazebo_sim/parts_descriptions/urdf/ScrewDriverBitStar.urdf (robot description, URDF)
Before this commit: robot ScrewDriverBitStar, 1 links, 0 joints
Links:
- link ScrewDriverBitStar: geometry collision mesh filename=package://rl_gazebo_sim/parts_descriptions/meshes/ScrewDriv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; visual mesh filename=package://rl_gazebo_sim/parts_descriptions/meshes/ScrewDriv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

File: rl_gazebo_sim/parts_descriptions/urdf/ScrewdriverBit(PZ2).urdf (robot description, URDF)
Before this commit: robot ScrewdriverBit(PZ2), 1 links, 0 joints
Links:
- link ScrewdriverBit(PZ2): geometry collision mesh filename=package://rl_gazebo_sim/parts_descriptions/meshes/Screwdriv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; visual mesh filename=package://rl_gazebo_sim/parts_descriptions/meshes/Screwdriv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
