Commit message: compleatly new assembly that's easier to understand

File: rl_gazebo_sim/parts_descriptions/screw_tool/screw_tool.urdf.xacro (robot description, xacro)
@@ -1,17 +1,18 @@
 <?xml version="2.0"?>
 <robot xmlns:xacro="http://ros.org/wiki/xacro">
-  <xacro:macro name="my_tool" params="parrent_link origin_xyz origin_rpy">
-    <!-- ft-sensor -->
-    <xacro:include filename="$(find rl_gazebo_sim)/parts_descriptions/urdf/ForceTorqueWithMount.urdf"/>
-    <!-- add the ft-senser -->
-    <joint name="${parrent_link}_ForceTorqueWithMount" type="revolute">
-      <origin xyz="${origin_xyz}" rpy="${origin_rpy}" />
-      <parent link="${parrent_link}"/>
-      <child link="ForceTorqueWithMount"/>
-      <axis xyz="0.0 0.0 1.0"/>
-      <limit velocity="6.5" effort="1000" lower="0" upper="0" />  <!--This is a bugfix. Using fixed type joint causes problems with FT-sensor.-->
+  <xacro:macro name="my_tool" params="prefix">
+    <!-- include the ft-sensor -->
+    <xacro:include filename="$(find rl_gazebo_sim)/parts_descriptions/urdf/ft_sensor.urdf"/>
+    <!-- Include the drill and mount -->
+    <xacro:include filename="$(find rl_gazebo_sim)/parts_descriptions/urdf/drill.urdf"/>
+    <!-- Add the drill to the ft_sensor -->
+    <joint name="ft_sensor_drill_joint" type="fixed">
+      <origin xyz="0 0 0.06342" rpy="0.0 0.0 ${pi/4}"/>
+      <parent link="ft_sensor"/>
+      <child link="drill"/>
     </joint>
-    <!-- Activate the feedback -->
-    <gazebo reference="${parrent_link}_ForceTorqueWithMount">
+    <!-- Activate the feedback and make sure the joint dont get reduced because it's fixed.-->
+    <gazebo reference="ft_sensor_drill_joint">
+      <disableFixedJointLumping>true</disableFixedJointLumping>
       <provideFeedback>true</provideFeedback>
     </gazebo>
@@ -22,34 +23,28 @@
         <topicName>FTsensor_topic</topicName>
         <gaussianNoise>0.0</gaussianNoise>
-        <jointName>${parrent_link}_ForceTorqueWithMount</jointName>
+        <jointName>ft_sensor_drill_joint</jointName>
       </plugin>
     </gazebo>
-    <!-- Drill and mount -->
-    <xacro:include filename="$(find rl_gazebo_sim)/parts_descriptions/urdf/DrillAndMountAssembly.urdf"/>
-    <!-- Add the drill to the chain -->
-    <joint name="ForceTorqueWithMount_DrillAndMountAssembly" type="fixed">
-      <origin xyz="0 -0.06342 0" rpy="0.0 ${pi/4} 0.0"/>
-      <parent link="ForceTorqueWithMount"/>
-      <child link="DrillAndMountAssembly"/>
-      <axis xyz="0.0 0.0 0.0"/>
-      <limit lower="0.0" upper="0.0" effort="0.0" velocity="0.0"/>
-    </joint>
     <!-- include the screw bit-->
     <xacro:include filename="$(find rl_gazebo_sim)/parts_descriptions/urdf/ScrewDriverBitStar.urdf"/>
     <!-- add the screw bit to the screw machine-->
-    <joint name="ForceTorqueWithMount_ScrewDriverBitStar" type="revolute">
-      <origin xyz="0 -0.22042 0" rpy="0 0 0" /> <!--sunken 5mm in to the bit holder -->
-      <parent link="ForceTorqueWithMount"/>
+    <joint name="drill_ScrewDriverBitStar_joint" type="revolute">
+      <origin xyz="0  0 0.147" rpy="0 0 0" /> <!--162mm but sunken 15mm in to the bit holder -->
+      <parent link="drill"/>
       <child link="ScrewDriverBitStar"/>
-      <axis xyz="0 1 0"/>
-      <limit velocity="1000" effort="1" lower="-100000000" upper="100000000"/>
+      <axis xyz="0 0 1"/>
+      <limit velocity="1000" effort="1" lower="-100" upper="100"/>
       </joint>
-    <!-- Frame coincident with all-zeros TCP on UR controller -->
+    <!-- Frame coincident with the tip of the screw driver bit -->
     <link name="ee_tip"/>
     <joint name="ScrewDriverBitStar_ee_tip" type="fixed">
-      <origin xyz="0 -0.025 0" rpy="${pi/-2.0} 0 0"/>
+      <origin xyz="0 0.025 0" rpy="0 0 0"/>
       <parent link="ScrewDriverBitStar"/>
       <child link="ee_tip"/>
-    </joint>
+      </joint>
+    <!--dont reduce the fixed joint -->
+    <gazebo reference="ee_tip">
+      <disableFixedJointLumping>true</disableFixedJointLumping>
+    </gazebo>
   </xacro:macro>
 </robot>

File: rl_gazebo_sim/ur5_robot_w_tool/ur5_robot_w_tool.urdf.xacro (robot description, xacro)
@@ -4,12 +4,23 @@
   <!-- common stuff -->
   <xacro:include filename="$(find ur_description)/urdf/common.gazebo.xacro" />
-  <!-- ur5 -->
+  <!-- include the ur5 -->
   <xacro:include filename="$(find ur_description)/urdf/ur5.urdf.xacro" />
-  <!-- tool -->
-  <xacro:include filename="$(find rl_gazebo_sim)/screw_tool/screw_tool.urdf.xacro" />
-  <!-- create the arm -->
+  <!-- include tool -->
+  <xacro:include filename="$(find rl_gazebo_sim)/parts_descriptions/screw_tool/screw_tool.urdf.xacro" />
+  <!-- create the arm macro-->
   <xacro:ur5_robot prefix="" joint_limited="true"/>
-  <!-- create the tool -->
-  <xacro:my_tool parrent_link="wrist_3_link" origin_xyz="0 0.0823 0" origin_rpy="${pi} ${pi/4} 0"/>
+  <!-- create the tool macro-->
+  <xacro:my_tool prefix=""/>
+  <!--dont reduce the fixed joint -->
+    <gazebo reference="ee_fixed_joint">
+      <disableFixedJointLumping>true</disableFixedJointLumping>
+    </gazebo>
+  <!-- add screw_tool to the robot -->
+    <joint name="ur_screw_tool_joint" type="fixed">
+      <origin xyz="0 0 0" rpy="0 ${pi/2} 0" />
+      <parent link="ee_link"/>
+      <child link="ft_sensor"/>
+    </joint>
+  <!-- Create a world link and fix it all to that -->
   <link name="world" />
   <!-- fix the arm in the world -->

Commit message: finalised the tool and robot + added a transmision interface to the screw tool

File: rl_gazebo_sim/parts_descriptions/screw_tool/screw_tool.urdf.xacro (robot description, xacro)
@@ -47,4 +47,18 @@
       <disableFixedJointLumping>true</disableFixedJointLumping>
     </gazebo>
+    <!--
+      add transmision to the screw_tool so it can be controlled by ros
+      it is added to the same hardware_interface as the ur robot so it
+      is the same namespace
+    -->
+    <transmission name="screw_tool_trans">
+      <type>transmission_interface/SimpleTransmission</type>
+      <joint name="drill_ScrewDriverBitStar_joint">
+        <hardwareInterface>hardware_interface/PositionJointInterface</hardwareInterface>
+      </joint>
+      <actuator name="screw_motor">
+        <mechanicalReduction>1</mechanicalReduction>
+      </actuator>
+    </transmission>
   </xacro:macro>
 </robot>

File: rl_gazebo_sim/ur5_robot_w_tool/ur5_robot_w_tool.urdf.xacro (robot description, xacro)
@@ -2,6 +2,11 @@
 <robot xmlns:xacro="http://ros.org/wiki/xacro"
        name="ur5" >
-  <!-- common stuff -->
-  <xacro:include filename="$(find ur_description)/urdf/common.gazebo.xacro" />
+  <!-- launch the ros_controller for gazebo that publishes the hardware interfaces -->
+  <gazebo>
+    <plugin name="ros_control" filename="libgazebo_ros_control.so">
+      <robotNamespace>/ur5</robotNamespace>
+      <!--robotSimType>gazebo_ros_control/DefaultRobotHWSim</robotSimType-->
+    </plugin>
+  </gazebo>
   <!-- include the ur5 -->
   <xacro:include filename="$(find ur_description)/urdf/ur5.urdf.xacro" />

Commit message: updating the screw to a new version

File: rl_gazebo_sim/parts_descriptions/screw_tool/screw_tool.urdf.xacro (robot description, xacro)
@@ -39,5 +39,5 @@
     <link name="ee_tip"/>
     <joint name="ScrewDriverBitStar_ee_tip" type="fixed">
-      <origin xyz="0 0.025 0" rpy="0 0 0"/>
+      <origin xyz="0 0 0.025" rpy="0 0 0"/>
       <parent link="ScrewDriverBitStar"/>
       <child link="ee_tip"/>

Commit message: minor name changes

File: rl_gazebo_sim/parts_descriptions/screw_tool/screw_tool.urdf.xacro (robot description, xacro)
@@ -1,5 +1,6 @@
 <?xml version="2.0"?>
 <robot xmlns:xacro="http://ros.org/wiki/xacro">
-  <xacro:macro name="my_tool" params="prefix">
+  <!-- A macro to create a screw tool. The param "prefix" is not yet implemented -->
+  <xacro:macro name="screw_tool" params="prefix">
     <!-- include the ft-sensor -->
     <xacro:include filename="$(find rl_gazebo_sim)/parts_descriptions/screw_tool/ft_sensor.urdf"/>

File: rl_gazebo_sim/ur5_robot_w_tool/ur5_robot_w_tool.urdf.xacro (robot description, xacro)
@@ -16,5 +16,5 @@
   <xacro:ur5_robot prefix="" joint_limited="true"/>
   <!-- create the tool macro-->
-  <xacro:my_tool prefix=""/>
+  <xacro:screw_tool prefix=""/>
   <!--dont reduce the fixed joint -->
     <gazebo reference="ee_fixed_joint">

Commit message: changed maximum value for turns on the screw bit from 100 to 1000

File: rl_gazebo_sim/parts_descriptions/screw_tool/screw_tool.urdf.xacro (robot description, xacro)
@@ -35,5 +35,5 @@
       <child link="ScrewDriverBitStar"/>
       <axis xyz="0 0 1"/>
-      <limit velocity="1000" effort="1" lower="-100" upper="100"/>
+      <limit velocity="1000" effort="1" lower="-1000" upper="1000"/>
       </joint>
     <!-- Frame coincident with the tip of the screw driver bit -->
@@ -56,5 +56,5 @@
       <type>transmission_interface/SimpleTransmission</type>
       <joint name="drill_ScrewDriverBitStar_joint">
-        <hardwareInterface>hardware_interface/PositionJointInterface</hardwareInterface>
+        <hardwareInterface>hardware_interface/VelocityJointInterface</hardwareInterface>
       </joint>
       <actuator name="screw_motor">
